File: hw/sch_pcb/LION1CELL02A.kicad_sch (KiCad schematic)
At the start: 82 parts

Commit message: minor changes
Parts:
- removed H? (x4): MountingHole_Pad, symbol Mechanical:MountingHole_Pad
- added M1, M2: HOLE M3, Mlab_Mechanical:MountingHole_3mm, symbol mlab-default-rescue:HOLE
- added M3, M4: HOLE, Mlab_Mechanical:MountingHole_3mm, symbol mlab-default-rescue:HOLE
- C1, C14, C5: renamed from C?; footprint (none) -> Mlab_C:SMD-0805
- C10, C11, C12, C13, C3, C4, C6, C7, C9: renamed from C?; footprint Mlab_R:SMD-0805 -> Mlab_C:SMD-0805
- C2: renamed from C?; footprint (none) -> Mlab_C:TantalC_SizeD_Reflow
- IC1: renamed from IC?; footprint SON65P200X200X80-7N -> (none)
- gave numbers to parts that had none: 64
Connections:
- net GND: now also M1.1, M2.1, M3.1, M4.1
Other:
- note added: "MOUNTING HOLES"
- note removed: "Mounting holes"
