File: hw/sch_pcb/LION1CELL02.kicad_sch (KiCad schematic)
At the start: 92 parts, among them J1 USBC_USB4105-GF-A, J2 HEADER_2x03, J3 HEADER_1x04, Q1 BSS83P, Q2 BC807-25, Q3 BC807-25, SW1 SKRTLAE010, U1 BQ34Z100, U2 BQ25628E, U3 TPS631000DRLR, U4 SN74HC164P, U5 BQ29700DSER

Commit message: Battery protection update
Parts:
- removed R28, R29: 4M7, Resistor_SMD:R_0805_2012Metric, symbol Device:R_Small
Changed lines of the file:
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@@
 	)
 	(junction
-		(at 218.44 233.68)
-		(diameter 0)
-		(color 0 0 0 0)
-	)
-	(junction
-		(at 213.36 220.98)
-		(diameter 0)
-		(color 0 0 0 0)
-	)
-	(junction
 		(at 229.87 189.23)
 		(diameter 0)
@@
 	)
 	(junction
-		(at 195.58 233.68)
-		(diameter 0)
-		(color 0 0 0 0)
-	)
-	(junction
 		(at 242.57 220.98)
 		(diameter 0)
@@
 	)
 	(junction
-		(at 200.66 220.98)
-		(diameter 0)
-		(color 0 0 0 0)
-	)
-	(junction
 		(at 314.96 217.17)
 		(diameter 0)
@@
 	(wire
 		(pts
-			(xy 195.58 229.87) (xy 195.58 233.68)
-		)
-		(stroke
-			(width 0)
-			(type default)
-		)
-	)
-	(wire
-		(pts
 			(xy 45.72 233.68) (xy 46.99 233.68)
 		)
@@
 	(wire
 		(pts
-			(xy 218.44 220.98) (xy 218.44 224.79)
-		)
-		(stroke
-			(width 0)
-			(type default)
-		)
-	)
-	(wire
-		(pts
 			(xy 93.98 266.7) (xy 105.41 266.7)
 		)
@@
 	(wire
 		(pts
-			(xy 218.44 229.87) (xy 218.44 233.68)
-		)
-		(stroke
-			(width 0)
-			(type default)
-		)
-	)
-	(wire
-		(pts
 			(xy 326.39 148.59) (xy 330.2 148.59)
 		)
@@
 	(wire
 		(pts
-			(xy 200.66 220.98) (xy 195.58 220.98)
-		)
-		(stroke
-			(width 0)
-			(type default)
-		)
-	)
-	(wire
-		(pts
 			(xy 175.26 52.07) (xy 175.26 53.34)
 		)
@@
 	(wire
 		(pts
-			(xy 195.58 220.98) (xy 195.58 224.79)
-		)
-		(stroke
-			(width 0)
-			(type default)
-		)
-	)
-	(wire
-		(pts
 			(xy 299.72 106.68) (xy 299.72 105.41)
 		)
@@
 	(wire
 		(pts
-			(xy 213.36 220.98) (xy 218.44 220.98)
-		)
-		(stroke
-			(width 0)
-			(type default)
-		)
-	)
-	(wire
-		(pts
 			(xy 173.99 189.23) (xy 229.87 189.23)
 		)
@@
 	)
 	(symbol
-		(lib_id "Device:R_Small")
-		(at 195.58 227.33 180)
-		(unit 1)
-		(exclude_from_sim no)
-		(in_bom yes)
-		(on_board yes)
-		(dnp no)
-		(property "Reference" "R28"
-			(at 193.294 226.568 0)
-			(effects
-				(font
-					(size 1 1)
-				)
-			)
-		)
-		(property "Value" "4M7"
-			(at 193.04 228.092 0)
-			(effects
-				(font
-					(size 1 1)
-				)
-			)
-		)
-		(property "Footprint" "Resistor_SMD:R_0805_2012Metric"
-			(at 195.58 227.33 0)
-			(effects
-				(font
-					(size 1 1)
-				)
-				(hide yes)
-			)
-		)
-		(property "Datasheet" "~"
-			(at 195.58 227.33 0)
-			(effects
-				(font
-					(size 1 1)
-				)
-				(hide yes)
-			)
-		)
-		(property "Description" "Resistor, small symbol"
-			(at 195.58 227.33 0)
-			(effects
-				(font
-					(size 1.27 1.27)
-				)
-				(hide yes)
-			)
-		)
-		(property "UST_ID" "5c70984512875079b91f8983"
-			(at 195.58 227.33 0)
-			(effects
-				(font
-					(size 1.27 1.27)
-				)
-				(hide yes)
-			)
-		)
-		(pin "1"
-		)
-		(pin "2"
-		)
-		(instances
-			(project "LION1CELL02"
-				(path "/949a5bba-1f1f-4325-9d02-2c6814a96048"
-					(reference "R28")
-					(unit 1)
-				)
-			)
-		)
-	)
-	(symbol
 		(lib_id "Device:C_Small")
 		(at 328.93 78.74 0)
@@
 					(unit 1)
 				)
-			)
-		)
-	)
-	(symbol
-		(lib_id "Device:R_Small")
-		(at 218.44 227.33 180)
-		(unit 1)
-		(exclude_from_sim no)
-		(in_bom yes)
-		(on_board yes)
-		(dnp no)
-		(property "Reference" "R29"
-			(at 220.98 226.568 0)
-			(effects
-				(font
-					(size 1 1)
-				)
-			)
-		)
-		(property "Value" "4M7"
-			(at 220.98 228.092 0)
-			(effects
-				(font
-					(size 1 1)
-				)
-			)
-		)
-		(property "Footprint" "Resistor_SMD:R_0805_2012Metric"
-			(at 218.44 227.33 0)
-			(effects
-				(font
-					(size 1 1)
-				)
-				(hide yes)
-			)
-		)
-		(property "Datasheet" "~"
-			(at 218.44 227.33 0)
-			(effects
-				(font
-					(size 1 1)
-				)
-				(hide yes)
-			)
-		)
-		(property "Description" "Resistor, small symbol"
-			(at 218.44 227.33 0)
-			(effects
-				(font
-					(size 1.27 1.27)
-				)
-				(hide yes)
-			)
-		)
-		(property "UST_ID" "5c70984512875079b91f8983"
-			(at 218.44 227.33 0)
-			(effects
-				(font
-					(size 1.27 1.27)
-				)
-				(hide yes)
-			)
-		)
-		(pin "1"
-		)
-		(pin "2"
-		)
-		(instances
-			(project "LION1CELL02"
-				(path "/949a5bba-1f1f-4325-9d02-2c6814a96048"
-					(reference "R29")
-					(unit 1)
-				)

Commit message: Update pcb
Connections:
- net -BAT: no longer U5.4 (VSS)
- net GND: no longer C19.2
- net at Q5.1 (G): now also U5.3 (Dout); no longer U5.2 (Cout)
- net at NT2.2, Q5.3 (S), R26.2: now also C19.2, U5.4 (VSS)
- net at Q4.1 (G): now also U5.2 (Cout); no longer U5.3 (Dout)
Other:
- moved on the sheet: BT1A, BT1B, C19, F1, F2, NT1, NT2, Q4, Q5, R25, R26, R27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

Commit message: Update sch
Parts:
- Q4, Q5: value ~ -> SI2302A-TP; footprint (none) -> Package_TO_SOT_SMD:SOT-23-3
- R25, R27: footprint (none) -> Resistor_SMD:R_0805_2012Metric
Other:
- note added: "Need to obtain 2.5 V"
- note removed: "Need to obtain 2.5V, here"
Changed lines of the file:
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@@
 		)
 	)
-	(text "Need to obtain 2.5V, here"
+	(text "Need to obtain 2.5 V\n"
 		(exclude_from_sim no)
 		(at 199.39 139.7 0)
@@
 			)
 		)
-		(property "Value" "~"
-			(at 209.55 244.856 0)
+		(property "Value" "SI2302A-TP"
+			(at 212.344 239.268 90)
 			(effects
 				(font
 					(size 1.27 1.27)
 				)
-				(hide yes)
 			)
 		)
-		(property "Footprint" ""
+		(property "Footprint" "Package_TO_SOT_SMD:SOT-23-3"
 			(at 208.28 236.22 0)
 			(effects
@@
 			)
 		)
-		(property "Footprint" ""
+		(property "Footprint" "Resistor_SMD:R_0805_2012Metric"
 			(at 224.79 198.12 0)
 			(effects
@@
 			)
 		)
-		(property "Footprint" ""
+		(property "Footprint" "Resistor_SMD:R_0805_2012Metric"
 			(at 187.96 224.79 0)
 			(effects
@@
 			)
 		)
-		(property "Value" "~"
-			(at 196.8501 237.49 0)
+		(property "Value" "SI2302A-TP"
+			(at 192.024 239.522 90)
 			(effects
 				(font
@@
 				)
 				(justify left)
-				(hide yes)
 			)
 		)
-		(property "Footprint" ""
+		(property "Footprint" "Package_TO_SOT_SMD:SOT-23-3"
 			(at 200.66 236.22 0)
 			(effects
