File: hw/sch_pcb/LION1CELL02.kicad_pcb (KiCad board)
At the start: 2 copper layers, 0 parts

Commit message: Update sch
Parts:
- added BT1: BATT, Mlab_Batery:BAT_BK-18650-PC4, F.Cu at (134.5, 65.6)
- added C1: 100n, Capacitor_SMD:C_0805_2012Metric, F.Cu at (119.9, 97.8)
- added C10: 10u, Capacitor_SMD:C_0805_2012Metric, F.Cu at (124.3, 103.8)
- added C11: 100n, Capacitor_SMD:C_0805_2012Metric, F.Cu at (124.3, 106.8)
- added C12: 3n3, Capacitor_SMD:C_0805_2012Metric, F.Cu at (124.3, 109.8)
- added C13: 1u, Capacitor_SMD:C_0805_2012Metric, F.Cu at (124.3, 112.8)
- added C14: 100n, Capacitor_SMD:C_0805_2012Metric, F.Cu at (124.3, 115.8)
- added C15: 22u, Capacitor_SMD:C_0805_2012Metric, F.Cu at (128.8, 97.8)
- added C16: 47u, Capacitor_SMD:C_0805_2012Metric, F.Cu at (128.8, 100.8)
- added C17: 10u, Capacitor_SMD:C_0805_2012Metric, F.Cu at (128.8, 103.8)
- added C18: 100n, Capacitor_SMD:C_0805_2012Metric, F.Cu at (128.8, 106.8)
- added C19: 100n, Capacitor_SMD:C_0805_2012Metric, F.Cu at (128.8, 109.8)
- added C2: 100n, Capacitor_SMD:C_0805_2012Metric, F.Cu at (119.9, 100.8)
- added C3: 1n, Capacitor_SMD:C_0805_2012Metric, F.Cu at (119.9, 103.8)
- added C4: 100n, Capacitor_SMD:C_0805_2012Metric, F.Cu at (119.9, 106.8)
- added C5: 47n, Capacitor_SMD:C_0805_2012Metric, F.Cu at (119.9, 109.8)
- added C6: 22u, Capacitor_SMD:C_0805_2012Metric, F.Cu at (119.9, 112.8)
- added C7: 10u, Capacitor_SMD:C_0805_2012Metric, F.Cu at (119.9, 115.8)
- added C8: 1u, Capacitor_SMD:C_0805_2012Metric, F.Cu at (124.3, 97.8)
- added C9: 4u7, Capacitor_SMD:C_0805_2012Metric, F.Cu at (124.3, 100.8)
- added D1: RED, Mlab_D:SMD_LED_RIGHT_KINGBRIGHT_1605, F.Cu at (141.5, 98.0)
- added D10: GREEN, Mlab_D:SMD_LED_RIGHT_KINGBRIGHT_1605, F.Cu at (145.0, 109.0)
- added D2: RED, Mlab_D:SMD_LED_RIGHT_KINGBRIGHT_1605, F.Cu at (141.5, 100.8)
- added D3: ORANGE, Mlab_D:SMD_LED_RIGHT_KINGBRIGHT_1605, F.Cu at (141.5, 103.5)
- added D4: ORANGE, Mlab_D:SMD_LED_RIGHT_KINGBRIGHT_1605, F.Cu at (141.5, 106.3)
- added D5: GREEN, Mlab_D:SMD_LED_RIGHT_KINGBRIGHT_1605, F.Cu at (141.5, 109.0)
- added D6: GREEN, Mlab_D:SMD_LED_RIGHT_KINGBRIGHT_1605, F.Cu at (145.0, 98.0)
- added D7: GREEN, Mlab_D:SMD_LED_RIGHT_KINGBRIGHT_1605, F.Cu at (145.0, 100.8)
- added D8: GREEN, Mlab_D:SMD_LED_RIGHT_KINGBRIGHT_1605, F.Cu at (145.0, 103.5)
- added D9: ORANGE, Mlab_D:SMD_LED_RIGHT_KINGBRIGHT_1605, F.Cu at (145.0, 106.3)
- added F1: Fuse, Fuse:Fuseholder_Littelfuse_Nano2_154x, F.Cu at (152.8, 111.8)
- added F2: Fuse, Fuse:Fuseholder_Littelfuse_Nano2_154x, F.Cu at (152.8, 118.4)
- added FID1: Fiducial, Fiducial:Fiducial_1mm_Mask2mm, F.Cu at (137.8, 92.6)
- added FID2: Fiducial, Fiducial:Fiducial_1mm_Mask2mm, F.Cu at (144.4, 92.6)
- added FID3: Fiducial, Fiducial:Fiducial_1mm_Mask2mm, F.Cu at (148.5, 92.5)
- added FID4: Fiducial, Fiducial:Fiducial_1mm_Mask2mm, F.Cu at (153.4, 91.8)
- added H1: M3, Mlab_Mechanical:MountingHole_3mm, F.Cu at (88.4, 40.9)
- added H2: M3, Mlab_Mechanical:MountingHole_3mm, F.Cu at (182.6, 88.1)
- added H3: M3, Mlab_Mechanical:MountingHole_3mm, F.Cu at (88.8, 88.6)
- added H4: M3, Mlab_Mechanical:MountingHole_3mm, F.Cu at (183.1, 40.6)
- added J1: USBC_USB4105-GF-A, Mlab_CON:USBC GCT_USB4105-GF-A, F.Cu at (101.2, 120.1)
- added J2: HEADER_2x03, Connector_PinHeader_2.54mm:PinHeader_2x03_P2.54mm_Vertical, F.Cu at (109.2, 116.3)
- added J3: HEADER_1x04, Connector_PinHeader_2.54mm:PinHeader_1x04_P2.54mm_Horizontal, F.Cu at (115.3, 127.6)
- added JP1: Jumper_3_Bridged12, Jumper:SolderJumper-3_P1.3mm_Bridged2Bar12_RoundedPad1.0x1.5mm, F.Cu at (136.2, 122.0)
- added L1: 1uH - DFE252012P-1R0M=P2, Inductor_SMD:L_1008_2520Metric, F.Cu at (162.6, 98.2)
- added L2: 1uH - DFE252012P-1R0M=P2, Inductor_SMD:L_1008_2520Metric, F.Cu at (162.6, 101.9)
- added NT1: NetTie_2, NetTie:NetTie-2_SMD_Pad0.5mm, F.Cu at (166.2, 104.5)
- added NT2: NetTie_2, NetTie:NetTie-2_SMD_Pad0.5mm, F.Cu at (166.2, 106.0)
- added Q1: BSS83P, Package_TO_SOT_SMD:SOT-23, F.Cu at (162.5, 106.0)
- added Q2: BC807-25, Package_TO_SOT_SMD:SOT-23-3, F.Cu at (133.6, 98.5)
- added Q3: BC807-25, Package_TO_SOT_SMD:SOT-23-3, F.Cu at (133.6, 103.0)
- added Q4: SI2302A-TP, Package_TO_SOT_SMD:SOT-23-3, F.Cu at (133.6, 107.4)
- added Q5: SI2302A-TP, Package_TO_SOT_SMD:SOT-23-3, F.Cu at (133.6, 111.9)
- added R1: 100R, Resistor_SMD:R_0805_2012Metric, F.Cu at (97.8, 97.8)
- added R10: 510R, Resistor_SMD:R_0805_2012Metric, F.Cu at (102.2, 106.6)
- added R11: 270R, Resistor_SMD:R_0805_2012Metric, F.Cu at (102.2, 109.6)
- added R12: 1k, Resistor_SMD:R_0805_2012Metric, F.Cu at (102.2, 112.5)
- added R13: 270R, Resistor_SMD:R_0805_2012Metric, F.Cu at (106.6, 97.8)
- added R14: 270R, Resistor_SMD:R_0805_2012Metric, F.Cu at (106.6, 100.7)
- added R15: 270R, Resistor_SMD:R_0805_2012Metric, F.Cu at (106.6, 103.7)
- added R16: 270R, Resistor_SMD:R_0805_2012Metric, F.Cu at (106.6, 106.6)
- added R17: 68R, Resistor_SMD:R_0805_2012Metric, F.Cu at (106.6, 109.6)
- added R18: 68R, Resistor_SMD:R_0805_2012Metric, F.Cu at (106.6, 112.5)
- added R19: 68R, Resistor_SMD:R_0805_2012Metric, F.Cu at (111.1, 97.8)
- added R2: 5k1, Resistor_SMD:R_0805_2012Metric, F.Cu at (97.8, 100.7)
- added R20: 68R, Resistor_SMD:R_0805_2012Metric, F.Cu at (111.1, 100.7)
- added R21: 1k, Resistor_SMD:R_0805_2012Metric, F.Cu at (111.1, 103.7)
- added R22: 1k, Resistor_SMD:R_0805_2012Metric, F.Cu at (111.1, 106.6)
- added R23: 270R, Resistor_SMD:R_0805_2012Metric, F.Cu at (111.1, 109.6)
- added R24: 68R, Resistor_SMD:R_0805_2012Metric, F.Cu at (111.1, 112.5)
- added R25: 330, Resistor_SMD:R_0805_2012Metric, F.Cu at (115.5, 97.8)
- added R26: 0R01 75PPM, Resistor_SMD:R_2512_6332Metric, F.Cu at (163.2, 117.7)
- added R27: 2k2, Resistor_SMD:R_0805_2012Metric, F.Cu at (115.5, 100.7)
- added R3: 5k1, Resistor_SMD:R_0805_2012Metric, F.Cu at (97.8, 103.7)
- added R30: 4k7, Resistor_SMD:R_0805_2012Metric, F.Cu at (115.5, 103.7)
- added R31: 4k7, Resistor_SMD:R_0805_2012Metric, F.Cu at (115.5, 106.6)
- added R4: 100R, Resistor_SMD:R_0805_2012Metric, F.Cu at (97.8, 106.6)
- added R5: 5k1, Resistor_SMD:R_0805_2012Metric, F.Cu at (97.8, 109.6)
- added R6: 33k, Resistor_SMD:R_0805_2012Metric, F.Cu at (97.8, 112.5)
- added R7: 2k4, Resistor_SMD:R_0805_2012Metric, F.Cu at (102.2, 97.8)
- added R8: 511k, Resistor_SMD:R_0805_2012Metric, F.Cu at (102.2, 100.7)
- added R9: 91k, Resistor_SMD:R_0805_2012Metric, F.Cu at (102.2, 103.7)
- added SW1: SKRTLAE010, Mlab_SW:SKRT, F.Cu at (143.0, 113.8)
- added TH1: 10k NTC, Resistor_SMD:R_0805_2012Metric, F.Cu at (115.5, 109.6)
- added TH2: 10k NTC, Resistor_SMD:R_0805_2012Metric, F.Cu at (115.5, 112.5)
- added U1: BQ34Z100, Mlab_IO:TSSOP-14_4.4x5mm_Pitch0.65mm, F.Cu at (122.1, 120.7)
- added U2: BQ25628E, Mlab_IO:Texas_S-WQFN-HR-18, F.Cu at (142.2, 121.7)
- added U3: TPS631000DRLR, Package_TO_SOT_SMD:SOT-583-8, F.Cu at (160.7, 122.1)
- added U4: SN74HC164P, Package_SO:TSSOP-14_4.4x5mm_P0.65mm, F.Cu at (163.3, 111.9)
- added U5: BQ29700DSER, Package_SON:WSON-6_1.5x1.5mm_P0.5mm, F.Cu at (164.3, 121.9)

Commit message: Pridani ochrany proti prehrati pres alert pin
Parts:
- moved J1 96.2 mm to (181.0, 66.3), turned to -90 degrees
- moved U1 11.4 mm to (110.7, 121.4)
- moved J3 9.54 mm to (105.9, 129.3)
- moved FID4 9.45 mm to (162.8, 90.8)
- moved U2 8.85 mm to (136.6, 128.5)
- moved J2 8.83 mm to (100.6, 118.4)
Changed lines of the file:
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@@
 	(footprint "Fiducial:Fiducial_1mm_Mask2mm"
 		(layer "F.Cu")
-		(at 153.416 91.821)
+		(at 162.814 90.805)
 		(descr "Fiducial, circular marking, 1mm bare copper, 2mm soldermask opening (Level A)")
 		(tags "fiducial")
@@
 	(footprint "Mlab_IO:Texas_S-WQFN-HR-18"
 		(layer "F.Cu")
-		(at 142.19026 121.66978)
+		(at 136.574 128.512)
 		(descr "20-Pin Plastic Quad Flatpack No-Lead Package, Body 3.0x3.0x0.8mm, Texas Instruments (http://www.ti.com/lit/ds/symlink/tps22993.pdf)")
 		(tags "QFN 0.4")
@@
 	(footprint "Mlab_IO:TSSOP-14_4.4x5mm_Pitch0.65mm"
 		(layer "F.Cu")
-		(at 122.14026 120.67978)
+		(at 110.744 121.412)
 		(descr "14-Lead Plastic Thin Shrink Small Outline (ST)-4.4 mm Body [TSSOP] (see Microchip Packaging Specification 00000049BS.pdf)")
 		(tags "SSOP 0.65")
@@
 	(footprint "Mlab_CON:USBC GCT_USB4105-GF-A"
 		(layer "F.Cu")
-		(at 101.24026 120.08978)
+		(at 180.975 66.294 -90)
 		(property "Reference" "J1"
-			(at -1.925 -6.335 0)
+			(at -1.925 -6.335 90)
 			(layer "F.SilkS")
 			(hide yes)
@@
 		)
 		(property "Value" "USBC_USB4105-GF-A"
-			(at 0.0625 3.735 0)
+			(at 0.0625 3.735 90)
 			(layer "F.Fab")
 			(hide yes)
@@
 		)
 		(property "Datasheet" ""
-			(at 0 0 0)
+			(at 0 0 90)
 			(layer "F.Fab")
 			(hide yes)
@@
 		)
 		(property "Description" "USB 2.0-only Type-C Receptacle connector"
-			(at 0 0 0)
+			(at 0 0 90)
 			(layer "F.Fab")
 			(hide yes)
@@
 		)
 		(property "MFPN" "USB4105-GF-A"
-			(at 0 0 0)
+			(at 0 0 270)
 			(unlocked yes)
 			(layer "F.Fab")
@@
 		)
 		(property "UST_ID" "5fa0f94612875025b397795e"
-			(at 0 0 0)
+			(at 0 0 270)
 			(unlocked yes)
 			(layer "F.Fab")
@@
 		)
 		(property "MPN" "USB4105-GF-A"
-			(at 0 0 0)
+			(at 0 0 270)
 			(unlocked yes)
 			(layer "F.Fab")
@@
 		(attr smd)
 		(fp_line
-			(start -4.79 -2.65)
-			(end -4.79 -1.4)
+			(start -4.79 2.6)
+			(end 4.79 2.6)
 			(stroke
 				(width 0.2)
@@
 		)
 		(fp_line
-			(start -4.79 1.32)
-			(end -4.79 2.6)
+			(start 4.79 2.6)
+			(end 4.79 1.32)
 			(stroke
 				(width 0.2)
@@
 		)
 		(fp_line
-			(start -4.79 2.6)
-			(end 4.79 2.6)
+			(start -4.79 1.32)
+			(end -4.79 2.6)
 			(stroke
 				(width 0.2)
@@
 		)
 		(fp_line
-			(start 4.79 -2.65)
-			(end 4.79 -1.4)
+			(start -4.79 -2.65)
+			(end -4.79 -1.4)
 			(stroke
 				(width 0.2)
@@
 		)
 		(fp_line
-			(start 4.79 2.6)
-			(end 4.79 1.32)
+			(start 4.79 -2.65)
+			(end 4.79 -1.4)
 			(stroke
 				(width 0.2)
@@
 		)
 		(fp_line
-			(start -5.1 -5.58)
-			(end -5.1 2.85)
+			(start -5.1 2.85)
+			(end 5.1 2.85)
 			(stroke
 				(width 0.05)
@@
 		)
 		(fp_line
-			(start -5.1 2.85)
-			(end 5.1 2.85)
+			(start 5.1 2.85)
+			(end 5.1 -5.58)
 			(stroke
 				(width 0.05)
@@
 		)
 		(fp_line
-			(start 5.1 -5.58)
-			(end -5.1 -5.58)
+			(start -5.1 -5.58)
+			(end -5.1 2.85)
 			(stroke
 				(width 0.05)
@@
 		)
 		(fp_line
-			(start 5.1 2.85)
-			(end 5.1 -5.58)
+			(start 5.1 -5.58)
+			(end -5.1 -5.58)
 			(stroke
 				(width 0.05)
@@
 		)
 		(fp_line
-			(start -4.79 -4.93)
-			(end 4.79 -4.93)
+			(start -4.79 2.6)
+			(end -4.79 -4.93)
 			(stroke
 				(width 0.1)
@@
 		)
 		(fp_line
-			(start -4.79 2.6)
-			(end -4.79 -4.93)
+			(start 4.79 2.6)
+			(end -4.79 2.6)
 			(stroke
 				(width 0.1)
@@
 		)
 		(fp_line
-			(start 4.79 -4.93)
-			(end 4.79 2.6)
+			(start -4.79 -4.93)
+			(end 4.79 -4.93)
 			(stroke
 				(width 0.1)
@@
 		)
 		(fp_line
-			(start 4.79 2.6)
-			(end -4.79 2.6)
+			(start 4.79 -4.93)
+			(end 4.79 2.6)
 			(stroke
 				(width 0.1)
@@
 		)
 		(pad "" np_thru_hole circle
-			(at -2.89 -3.68)
+			(at -2.89 -3.68 270)
 			(size 0.65 0.65)
 			(drill 0.65)
@@
 		)
 		(pad "" np_thru_hole circle
-			(at 2.89 -3.68)
+			(at 2.89 -3.68 270)
 			(size 0.65 0.65)
 			(drill 0.65)
@@
 		)
 		(pad "A1/B12" smd rect
-			(at -3.2 -4.755)
+			(at -3.2 -4.755 270)
 			(size 0.6 1.15)
 			(layers "F.Cu" "F.Mask" "F.Paste")
@@
 		)
 		(pad "A4/B9" smd rect
-			(at -2.4 -4.755)
+			(at -2.4 -4.755 270)
 			(size 0.6 1.15)
 			(layers "F.Cu" "F.Mask" "F.Paste")
@@
 		)
 		(pad "A5" smd rect
-			(at -1.25 -4.755)
+			(at -1.25 -4.755 270)
 			(size 0.3 1.15)
 			(layers "F.Cu" "F.Mask" "F.Paste")
@@
 		)
 		(pad "A6" smd rect
-			(at -0.25 -4.755)
+			(at -0.25 -4.755 270)
 			(size 0.3 1.15)
 			(layers "F.Cu" "F.Mask" "F.Paste")
@@
 		)
 		(pad "A7" smd rect
-			(at 0.25 -4.755)
+			(at 0.25 -4.755 270)
 			(size 0.3 1.15)
 			(layers "F.Cu" "F.Mask" "F.Paste")
@@
 		)
 		(pad "A8" smd rect
-			(at 1.25 -4.755)
+			(at 1.25 -4.755 270)
 			(size 0.3 1.15)
 			(layers "F.Cu" "F.Mask" "F.Paste")
@@
 		)
 		(pad "B1/A12" smd rect
-			(at 3.2 -4.755)
+			(at 3.2 -4.755 270)
 			(size 0.6 1.15)
 			(layers "F.Cu" "F.Mask" "F.Paste")
@@
 		)
 		(pad "B4/A9" smd rect
-			(at 2.4 -4.755)
+			(at 2.4 -4.755 270)
 			(size 0.6 1.15)
 			(layers "F.Cu" "F.Mask" "F.Paste")
@@
 		)
 		(pad "B5" smd rect
-			(at 1.75 -4.755)
+			(at 1.75 -4.755 270)
 			(size 0.3 1.15)
 			(layers "F.Cu" "F.Mask" "F.Paste")
@@
 		)
 		(pad "B6" smd rect
-			(at 0.75 -4.755)
+			(at 0.75 -4.755 270)
 			(size 0.3 1.15)
 			(layers "F.Cu" "F.Mask" "F.Paste")
@@
 		)
 		(pad "B7" smd rect
-			(at -0.75 -4.755)
+			(at -0.75 -4.755 270)
 			(size 0.3 1.15)
 			(layers "F.Cu" "F.Mask" "F.Paste")
@@
 		)
 		(pad "B8" smd rect
-			(at -1.75 -4.755)
+			(at -1.75 -4.755 270)
 			(size 0.3 1.15)
 			(layers "F.Cu" "F.Mask" "F.Paste")
@@
 		)
 		(pad "G1" thru_hole oval
-			(at -4.32 0)
+			(at -4.32 0 270)
 			(size 1 2)
 			(drill oval 0.6 1.4)
@@
 		)
 		(pad "G2" thru_hole oval
-			(at 4.32 0)
+			(at 4.32 0 270)
 			(size 1 2)
 			(drill oval 0.6 1.4)
@@
 		)
 		(pad "G3" thru_hole oval
-			(at -4.32 -4.18)
+			(at -4.32 -4.18 270)
 			(size 1.05 2.1)
 			(drill oval 0.6 1.7)
@@
 		)
 		(pad "G4" thru_hole oval
-			(at 4.32 -4.18)
+			(at 4.32 -4.18 270)
 			(size 1.05 2.1)
 			(drill oval 0.6 1.7)
@@
 	(footprint "Connector_PinHeader_2.54mm:PinHeader_2x03_P2.54mm_Vertical"
 		(layer "F.Cu")
-		(at 109.16026 116.27978)
+		(at 100.584 118.364)
 		(descr "Through hole straight pin header, 2x03, 2.54mm pitch, double rows")
 		(tags "Through hole pin header THT 2x03 2.54mm double row")
@@
 	(footprint "Connector_PinHeader_2.54mm:PinHeader_1x04_P2.54mm_Horizontal"
 		(layer "F.Cu")
-		(at 115.316 127.635 -90)
+		(at 105.918 129.286 -90)
 		(descr "Through hole angled pin header, 1x04, 2.54mm pitch, 6mm pin length, single row")
 		(tags "Through hole angled pin header THT 1x04 2.54mm single row")

Commit message: Update sch
Parts:
- added D11: BAT54C, Mlab_IO:SOT-23, F.Cu at (178.5, 110.1)
- added R28: 10k, Resistor_SMD:R_0805_2012Metric, F.Cu at (174.3, 109.5)
- added R29: 10k, Resistor_SMD:R_0805_2012Metric, F.Cu at (174.3, 112.4)
- Q4, Q5: value SI2302A-TP -> AO3400A
- moved U3 7.46 mm to (154.4, 126.1)
- moved U5 4.01 mm to (165.8, 125.6)
Connections:
- U1 pad 12: unconnected-(U1-P5/HDQ-Pad12) -> /ALERT
- U5 pad 2: Net-(Q4-G) -> Net-(U5-Cout)
- U5 pad 3: Net-(Q5-G) -> Net-(U5-Dout)

Commit message: Update pcb
Parts:
- C1, C10, C11, C12, C13, C14, C15, C16, C17, C18, C19, C2, C3, C4, C5, C6, C7, C8, C9, D11, F1, F2, J1, JP1, L1, L2, NT1, NT2, Q1, Q4, Q5, R1, R10, R11, R12, R2, R25, R26, R27, R3, R4, R5, R6, R7, R8, R9, TH1, TH2, U1, U2, U3, U4, U5: moved to B.Cu
- R28, R29: value 10k -> 1k; moved to B.Cu
- moved R3 137.7 mm to (227.2, 56.6)
- moved R2 137.3 mm to (227.2, 54.6)
- moved FID1 123.8 mm to (240.6, 161.5)
- moved FID2 123.8 mm to (247.2, 161.5)
- moved FID3 123.8 mm to (251.3, 161.4)
- moved C3 118.8 mm to (227.2, 52.7), turned to 180 degrees
- moved FID4 117.8 mm to (257.4, 161.0)
- moved Q1 102.1 mm to (70.3, 62.1)
- moved NT2 91.2 mm to (78.2, 81.8), turned to 180 degrees
- moved R26 89.0 mm to (80.8, 84.3), turned to 180 degrees
- moved L1 87.8 mm to (75.7, 110.9), turned to 90 degrees
- moved NT1 86.0 mm to (83.2, 81.8)
- moved J2 84.9 mm to (181.2, 145.0), turned to 90 degrees
- moved JP1 83.8 mm to (72.2, 67.8)
- moved R28 82.9 mm to (99.8, 73.2), turned to 90 degrees
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Connections:
- BT1 pad 1-: /-BAT -> Net-(BT1A--)
- BT1 pad 2-: /-BAT -> Net-(BT1A--)
- C19 pad 2: Net-(Q5-S) -> Net-(BT1A--)
- NT1 pad 2: /-BAT -> Net-(Q4-S)
- NT2 pad 2: Net-(Q5-S) -> GND
- Q4 pad 3: GND -> Net-(Q4-S)
- Q5 pad 3: Net-(Q5-S) -> Net-(BT1A--)
- R26 pad 1: /-BAT -> Net-(Q4-S)
- R26 pad 2: Net-(Q5-S) -> GND
- R27 pad 2: GND -> Net-(Q4-S)
- U5 pad 4: Net-(Q5-S) -> Net-(BT1A--)
